File: OpenA1200RTC.kicad_pcb (KiCad board)
At the start: 2 copper layers, 44.5 x 35.8 mm, 14 parts, among them J1 Connector_2x20_2mm, U1 MSM6242B

Commit message: Handsoldering footprint for D1
Parts:
- D1: footprint TO_SOT_Packages_SMD:SOT-23 -> TO_SOT_Packages_SMD:SOT-23_Handsoldering
- V1: footprint library:oshw -> library:OSHW
- moved V1 1.86 mm to (137.8, 85.9)
- moved D1 0.21 mm to (164.7, 81.5)
