File: OpenA1200RTC.sch (KiCad schematic (older format))
At the start: 14 parts, among them J1 Connector_2x20_2mm, U1 MSM6242B

Commit message: Handsoldering footprint for D1
Parts:
- D1: footprint TO_SOT_Packages_SMD:SOT-23 -> TO_SOT_Packages_SMD:SOT-23_Handsoldering
- V1: footprint library:oshw -> library:OSHW
Changed lines of the file:
@@
 F 0 "D1" H 6900 1975 50  0000 C CNN
 F 1 "BAT54C" H 6900 1884 50  0000 C CNN
-F 2 "TO_SOT_Packages_SMD:SOT-23" H 6975 1875 50  0001 L CNN
+F 2 "TO_SOT_Packages_SMD:SOT-23_Handsoldering" H 6975 1875 50  0001 L CNN
 F 3 "http://www.diodes.com/_files/datasheets/ds11005.pdf" H 6820 1750 50  0001 C CNN
 	1    6900 1750
@@
 F 0 "V1" H 10128 6296 50  0000 L CNN
 F 1 "OSHW" H 10128 6205 50  0000 L CNN
-F 2 "library:oshw" H 10050 6250 50  0001 C CNN
+F 2 "library:OSHW" H 10050 6250 50  0001 C CNN
 F 3 "" H 10050 6250 50  0001 C CNN
 	1    10050 6250
@@
 BAT721C \ns also fine
 $Comp
-L power:VDD #PWR?
+L power:VDD #PWR0111
 U 1 1 5C2FE349
 P 10450 950
-F 0 "#PWR?" H 10450 800 50  0001 C CNN
+F 0 "#PWR0111" H 10450 800 50  0001 C CNN
 F 1 "VDD" H 10467 1123 50  0000 C CNN
 F 2 "" H 10450 950 50  0001 C CNN
